File: zyno.kicad_pcb (KiCad board)
At the start: 2 copper layers, 3.4 x 3 mm, 76 parts, among them U1 RP2040_Pro_Micro

Commit message: Linked Schematic
Parts:
- removed REF** (x31): Choc_V1V2_1.00u, ScottoKeebs_Hotswap:Hotswap_Choc_V1V2_1.00u
- removed REF**: TRRS_PJ-320A, ScottoKeebs_Components:TRRS_PJ-320A
- removed REF**: RotaryEncoder_Alps_EC11E-Switch_Vertical_H20mm, Rotary_Encoder:RotaryEncoder_Alps_EC11E-Switch_Vertical_H20mm
- removed REF** (x3): Choc_V1V2_1.50u_90deg, ScottoKeebs_Hotswap:Hotswap_Choc_V1V2_1.50u_90deg
- removed REF**: LED_WS2812B, ScottoKeebs_Components:LED_WS2812B
- removed REF** (x34): 1N4148W, ScottoKeebs_Components:Diode_SOD-123
- removed REF** (x2): LED_SK6812MINI, ScottoKeebs_Components:LED_SK6812MINI
- removed REF**: Button_MJTP1243, ScottoKeebs_Components:Button_MJTP1243
- added D1: Diode, ScottoKeebs_Components:Diode_SOD-123, B.Cu at (45.4, 41.1)
- added D10: Diode, ScottoKeebs_Components:Diode_SOD-123, B.Cu at (102.4, 51.2)
- added D11: Diode, ScottoKeebs_Components:Diode_SOD-123, B.Cu at (120.4, 54.6)
- added D12: Diode, ScottoKeebs_Components:Diode_SOD-123, B.Cu at (138.4, 58.0)
- added D13: Diode, ScottoKeebs_Components:Diode_SOD-123, B.Cu at (46.6, 75.1)
- added D14: Diode, ScottoKeebs_Components:Diode_SOD-123, B.Cu at (64.6, 74.5)
- added D15: Diode, ScottoKeebs_Components:Diode_SOD-123, B.Cu at (84.4, 71.6)
- added D16: Diode, ScottoKeebs_Components:Diode_SOD-123, B.Cu at (102.4, 68.2)
- added D17: Diode, ScottoKeebs_Components:Diode_SOD-123, B.Cu at (120.4, 71.6)
- added D18: Diode, ScottoKeebs_Components:Diode_SOD-123, B.Cu at (138.4, 75.0)
- added D19: Diode, ScottoKeebs_Components:Diode_SOD-123, B.Cu at (47.2, 92.1)
- added D2: Diode, ScottoKeebs_Components:Diode_SOD-123, B.Cu at (63.4, 40.5)
- added D20: Diode, ScottoKeebs_Components:Diode_SOD-123, B.Cu at (65.2, 91.5)
- added D21: Diode, ScottoKeebs_Components:Diode_SOD-123, B.Cu at (84.4, 88.6)
- added D22: Diode, ScottoKeebs_Components:Diode_SOD-123, B.Cu at (102.4, 85.2)
- added D23: Diode, ScottoKeebs_Components:Diode_SOD-123, B.Cu at (120.4, 88.6)
- added D24: Diode, ScottoKeebs_Components:Diode_SOD-123, B.Cu at (138.4, 92.0)
- added D25: Diode, ScottoKeebs_Components:Diode_SOD-123, B.Cu at (157.7, 94.2)
- added D26: Diode, ScottoKeebs_Components:Diode_SOD-123, B.Cu at (176.9, 98.2)
- added D27: Diode, ScottoKeebs_Components:Diode_SOD-123, B.Cu at (47.8, 109.1)
- added D28: Diode, ScottoKeebs_Components:Diode_SOD-123, B.Cu at (65.8, 108.4)
- added D29: Diode, ScottoKeebs_Components:Diode_SOD-123, B.Cu at (84.4, 105.6)
- added D3: Diode, ScottoKeebs_Components:Diode_SOD-123, B.Cu at (84.4, 37.6)
- added D30: Diode, ScottoKeebs_Components:Diode_SOD-123, B.Cu at (120.4, 105.6)
- added D31: Diode, ScottoKeebs_Components:Diode_SOD-123, B.Cu at (137.9, 116.3)
- added D32: Diode, ScottoKeebs_Components:Diode_SOD-123, B.Cu at (156.9, 120.4)
- added D33: Diode, ScottoKeebs_Components:Diode_SOD-123, B.Cu at (175.5, 128.0)
- added D34: Diode, ScottoKeebs_Components:Diode_SOD-123, B.Cu at (90.8, 94.0)
- added D35: LED_SK6812MINI, ScottoKeebs_Components:LED_SK6812MINI, B.Cu at (39.8, 41.9)
- added D36: LED_SK6812MINI, ScottoKeebs_Components:LED_SK6812MINI, B.Cu at (57.8, 41.3)
- added D37: LED_SK6812MINI, ScottoKeebs_Components:LED_SK6812MINI, B.Cu at (78.8, 38.2)
- added D38: LED_SK6812MINI, ScottoKeebs_Components:LED_SK6812MINI, B.Cu at (96.8, 34.8)
- added D39: LED_SK6812MINI, ScottoKeebs_Components:LED_SK6812MINI, B.Cu at (114.8, 38.2)
- added D4: Diode, ScottoKeebs_Components:Diode_SOD-123, B.Cu at (102.4, 34.2)
- added D40: LED_SK6812MINI, ScottoKeebs_Components:LED_SK6812MINI, B.Cu at (132.8, 41.6)
- added D41: LED_SK6812MINI, ScottoKeebs_Components:LED_SK6812MINI, B.Cu at (40.4, 58.9)
- added D42: LED_SK6812MINI, ScottoKeebs_Components:LED_SK6812MINI, B.Cu at (58.4, 58.3)
- added D43: LED_SK6812MINI, ScottoKeebs_Components:LED_SK6812MINI, B.Cu at (78.8, 55.2)
- added D44: LED_SK6812MINI, ScottoKeebs_Components:LED_SK6812MINI, B.Cu at (96.8, 51.8)
- added D45: LED_SK6812MINI, ScottoKeebs_Components:LED_SK6812MINI, B.Cu at (114.8, 55.2)
- added D46: LED_SK6812MINI, ScottoKeebs_Components:LED_SK6812MINI, B.Cu at (132.8, 58.6)
- added D47: LED_SK6812MINI, ScottoKeebs_Components:LED_SK6812MINI, B.Cu at (41.0, 75.9)
- added D48: LED_SK6812MINI, ScottoKeebs_Components:LED_SK6812MINI, B.Cu at (58.9, 75.3)
- added D49: LED_SK6812MINI, ScottoKeebs_Components:LED_SK6812MINI, B.Cu at (78.8, 72.2)
- added D5: Diode, ScottoKeebs_Components:Diode_SOD-123, B.Cu at (120.4, 37.6)
- added D50: LED_SK6812MINI, ScottoKeebs_Components:LED_SK6812MINI, B.Cu at (96.8, 68.8)
- added D51: LED_SK6812MINI, ScottoKeebs_Components:LED_SK6812MINI, B.Cu at (114.8, 72.2)
- added D52: LED_SK6812MINI, ScottoKeebs_Components:LED_SK6812MINI, B.Cu at (132.8, 75.6)
- added D53: LED_SK6812MINI, ScottoKeebs_Components:LED_SK6812MINI, B.Cu at (41.5, 92.9)
- added D54: LED_SK6812MINI, ScottoKeebs_Components:LED_SK6812MINI, B.Cu at (59.5, 92.3)
- added D55: LED_SK6812MINI, ScottoKeebs_Components:LED_SK6812MINI, B.Cu at (78.8, 89.2)
- added D56: LED_SK6812MINI, ScottoKeebs_Components:LED_SK6812MINI, B.Cu at (96.8, 85.8)
- added D57: LED_SK6812MINI, ScottoKeebs_Components:LED_SK6812MINI, B.Cu at (114.8, 89.2)
- added D58: LED_SK6812MINI, ScottoKeebs_Components:LED_SK6812MINI, B.Cu at (132.8, 92.6)
- added D59: LED_SK6812MINI, ScottoKeebs_Components:LED_SK6812MINI, B.Cu at (152.0, 94.3)
- added D6: Diode, ScottoKeebs_Components:Diode_SOD-123, B.Cu at (138.4, 41.0)
- added D60: LED_SK6812MINI, ScottoKeebs_Components:LED_SK6812MINI, B.Cu at (171.3, 97.6)
- added D61: LED_SK6812MINI, ScottoKeebs_Components:LED_SK6812MINI, B.Cu at (42.1, 109.9)
- added D62: LED_SK6812MINI, ScottoKeebs_Components:LED_SK6812MINI, B.Cu at (60.1, 109.3)
- added D63: LED_SK6812MINI, ScottoKeebs_Components:LED_SK6812MINI, B.Cu at (78.8, 106.2)
- added D64: LED_SK6812MINI, ScottoKeebs_Components:LED_SK6812MINI, B.Cu at (114.8, 106.2)
- added D65: LED_SK6812MINI, ScottoKeebs_Components:LED_SK6812MINI, B.Cu at (132.2, 116.4)
- added D66: LED_SK6812MINI, ScottoKeebs_Components:LED_SK6812MINI, B.Cu at (151.3, 119.6)
- added D67: LED_SK6812MINI, ScottoKeebs_Components:LED_SK6812MINI, B.Cu at (170.1, 126.1)
- added D7: Diode, ScottoKeebs_Components:Diode_SOD-123, B.Cu at (46.0, 58.1)
- added D8: Diode, ScottoKeebs_Components:Diode_SOD-123, B.Cu at (64.0, 57.5)
- added D9: Diode, ScottoKeebs_Components:Diode_SOD-123, B.Cu at (84.4, 54.6)
- added D98: LED_WS2812B, ScottoKeebs_Components:LED_WS2812B, F.Cu at (215.3, 30.3)
- added S1: Keyswitch, ScottoKeebs_Hotswap:Hotswap_Choc_V1V2_1.00u, F.Cu at (39.6, 36.8)
- added S10: Keyswitch, ScottoKeebs_Hotswap:Hotswap_Choc_V1V2_1.00u, F.Cu at (96.8, 46.7)
- added S11: Keyswitch, ScottoKeebs_Hotswap:Hotswap_Choc_V1V2_1.00u, F.Cu at (114.8, 50.1)
- added S12: Keyswitch, ScottoKeebs_Hotswap:Hotswap_Choc_V1V2_1.00u, F.Cu at (132.8, 53.5)
- added S13: Keyswitch, ScottoKeebs_Hotswap:Hotswap_Choc_V1V2_1.00u, F.Cu at (40.8, 70.8)
- added S14: Keyswitch, ScottoKeebs_Hotswap:Hotswap_Choc_V1V2_1.00u, F.Cu at (58.8, 70.2)
- added S15: Keyswitch, ScottoKeebs_Hotswap:Hotswap_Choc_V1V2_1.00u, F.Cu at (78.8, 67.1)
- added S16: Keyswitch, ScottoKeebs_Hotswap:Hotswap_Choc_V1V2_1.00u, F.Cu at (96.8, 63.7)
- added S17: Keyswitch, ScottoKeebs_Hotswap:Hotswap_Choc_V1V2_1.00u, F.Cu at (114.8, 67.1)
- added S18: Keyswitch, ScottoKeebs_Hotswap:Hotswap_Choc_V1V2_1.00u, F.Cu at (132.8, 70.5)
- added S19: Keyswitch, ScottoKeebs_Hotswap:Hotswap_Choc_V1V2_1.00u, F.Cu at (41.4, 87.8)
- added S2: Keyswitch, ScottoKeebs_Hotswap:Hotswap_Choc_V1V2_1.00u, F.Cu at (57.6, 36.2)
- added S20: Keyswitch, ScottoKeebs_Hotswap:Hotswap_Choc_V1V2_1.00u, F.Cu at (59.4, 87.2)
- added S21: Keyswitch, ScottoKeebs_Hotswap:Hotswap_Choc_V1V2_1.00u, F.Cu at (78.8, 84.1)
- added S22: Keyswitch, ScottoKeebs_Hotswap:Hotswap_Choc_V1V2_1.00u, F.Cu at (96.8, 80.7)
- added S23: Keyswitch, ScottoKeebs_Hotswap:Hotswap_Choc_V1V2_1.00u, F.Cu at (114.8, 84.1)
- added S24: Keyswitch, ScottoKeebs_Hotswap:Hotswap_Choc_V1V2_1.00u, F.Cu at (132.8, 87.5)
- added S25: Keyswitch, ScottoKeebs_Hotswap:Hotswap_Choc_V1V2_1.00u, F.Cu at (152.6, 89.2)
- added S26: Keyswitch, ScottoKeebs_Hotswap:Hotswap_Choc_V1V2_1.00u, F.Cu at (172.4, 92.6)
- added S27: Keyswitch, ScottoKeebs_Hotswap:Hotswap_Choc_V1V2_1.00u, F.Cu at (42.0, 104.8)
- added S28: Keyswitch, ScottoKeebs_Hotswap:Hotswap_Choc_V1V2_1.00u, F.Cu at (60.0, 104.2)
- added S29: Keyswitch, ScottoKeebs_Hotswap:Hotswap_Choc_V1V2_1.00u, F.Cu at (78.8, 101.1)
- added S3: Keyswitch, ScottoKeebs_Hotswap:Hotswap_Choc_V1V2_1.00u, F.Cu at (78.8, 33.1)
- added S30: Keyswitch, ScottoKeebs_Hotswap:Hotswap_Choc_V1V2_1.00u, F.Cu at (114.8, 101.1)
- added S31: Keyswitch, ScottoKeebs_Hotswap:Hotswap_Choc_V1V2_1.50u_90deg, F.Cu at (132.8, 111.3)
- added S32: Keyswitch, ScottoKeebs_Hotswap:Hotswap_Choc_V1V2_1.50u_90deg, F.Cu at (152.6, 114.7)
- added S33: Keyswitch, ScottoKeebs_Hotswap:Hotswap_Choc_V1V2_1.50u_90deg, F.Cu at (172.4, 121.5)
- added S4: Keyswitch, ScottoKeebs_Hotswap:Hotswap_Choc_V1V2_1.00u, F.Cu at (96.8, 29.7)
- added S5: Keyswitch, ScottoKeebs_Hotswap:Hotswap_Choc_V1V2_1.00u, F.Cu at (114.8, 33.1)
- added S6: Keyswitch, ScottoKeebs_Hotswap:Hotswap_Choc_V1V2_1.00u, F.Cu at (132.8, 36.5)
- added S7: Keyswitch, ScottoKeebs_Hotswap:Hotswap_Choc_V1V2_1.00u, F.Cu at (40.2, 53.8)
- added S8: Keyswitch, ScottoKeebs_Hotswap:Hotswap_Choc_V1V2_1.00u, F.Cu at (58.2, 53.2)
- added S9: Keyswitch, ScottoKeebs_Hotswap:Hotswap_Choc_V1V2_1.00u, F.Cu at (78.8, 50.1)
- added SW1: Switch, ScottoKeebs_Components:Button_MJTP1243, F.Cu at (147.5, 73.5)
- added SW2: RotaryEncoder_Switch, Rotary_Encoder:RotaryEncoder_Alps_EC11E-Switch_Vertical_H20mm, F.Cu at (94.3, 106.9)
- added U2: TRRS, ScottoKeebs_Components:TRRS_PJ-320A, F.Cu at (172.4, 75.6)
- moved U1 22.2 mm to (161.6, 48.4)
- moved J1 20.9 mm to (177.7, 67.0)
- renumbered REF** to J1
Connections:
- J1 pad 1: (no net) -> unconnected-(J1-GND-Pad1)
- J1 pad 2: (no net) -> unconnected-(J1-VCC-Pad2)
- J1 pad 3: (no net) -> unconnected-(J1-SCL-Pad3)
- J1 pad 4: (no net) -> unconnected-(J1-SDA-Pad4)
- U1 pad 1: (no net) -> unconnected-(U1-GP10-Pad1)
- U1 pad 10: (no net) -> unconnected-(U1-GP6-Pad10)
- U1 pad 11: (no net) -> unconnected-(U1-GP7-Pad11)
- U1 pad 12: (no net) -> unconnected-(U1-GP8-Pad12)
- U1 pad 13: (no net) -> unconnected-(U1-GP9-Pad13)
- U1 pad 14: (no net) -> unconnected-(U1-GP12-Pad14)
- U1 pad 15: (no net) -> unconnected-(U1-GP13-Pad15)
- U1 pad 16: (no net) -> unconnected-(U1-GP14-Pad16)
- U1 pad 17: (no net) -> unconnected-(U1-GP15-Pad17)
- U1 pad 18: (no net) -> unconnected-(U1-GP16-Pad18)
- U1 pad 19: (no net) -> unconnected-(U1-GP21-Pad19)
- U1 pad 2: (no net) -> unconnected-(U1-GP0-Pad2)
- U1 pad 20: (no net) -> unconnected-(U1-GP23-Pad20)
- U1 pad 21: (no net) -> unconnected-(U1-GP20-Pad21)
- U1 pad 22: (no net) -> unconnected-(U1-GP22-Pad22)
- U1 pad 23: (no net) -> unconnected-(U1-GP26-Pad23)
- U1 pad 24: (no net) -> unconnected-(U1-GP27-Pad24)
- U1 pad 25: (no net) -> unconnected-(U1-GP28-Pad25)
- U1 pad 26: (no net) -> unconnected-(U1-GP29-Pad26)
- U1 pad 27: (no net) -> unconnected-(U1-3.3v-Pad27)
- U1 pad 28: (no net) -> unconnected-(U1-RST-Pad28)
- U1 pad 29: (no net) -> unconnected-(U1-GND-Pad29)
- U1 pad 3: (no net) -> /Row0
- U1 pad 30: (no net) -> unconnected-(U1-5v-Pad30)
- U1 pad 31: (no net) -> unconnected-(U1-GP11-Pad31)
- U1 pad 4: (no net) -> unconnected-(U1-GND-Pad4)
- U1 pad 5: (no net) -> unconnected-(U1-GND-Pad5)
- U1 pad 6: (no net) -> unconnected-(U1-GP2-Pad6)
- U1 pad 7: (no net) -> unconnected-(U1-GP3-Pad7)
- U1 pad 8: (no net) -> unconnected-(U1-GP4-Pad8)
- U1 pad 9: (no net) -> unconnected-(U1-GP5-Pad9)
Routing:
- net (no net): track 832.8 -> 0.00 mm, vias 6 -> 0
Other:
- board size 3.4 x 3 mm -> 4.4 x 4.2 mm
