File: zyno.kicad_sch (KiCad schematic)
At the start: 10 parts, among them J1 OLED_128x32, SW1 RotaryEncoder_Switch, SW2 Switch, U1 TRRS, U2 RP2040_Pro_Micro

Commit message: Linked Schematic
Parts:
- added D10, D11, D12, D13, D14, D15, D16, D17, D18, D19, D20, D21, D22, D23, D24, D25, D26, D27, D28, D29, D3, D30, D31, D32, D33, D34, D4, D5, D6, D7, D8, D9: Diode, ScottoKeebs_Components:Diode_SOD-123, symbol ScottoKeebs:Placeholder_Diode
- added D35, D36, D37, D38, D39, D40, D41, D42, D43, D44, D45, D46, D47, D48, D49, D50, D51, D52, D53, D54, D55, D56, D57, D58, D59, D60, D61, D62, D63, D64, D65, D66, D67: LED_SK6812MINI, ScottoKeebs_Components:LED_SK6812MINI, symbol ScottoKeebs:LED_SK6812MINI
- added S10, S11, S12, S13, S14, S15, S16, S17, S18, S19, S20, S21, S22, S23, S24, S25, S26, S27, S28, S29, S3, S30, S4, S5, S6, S7, S8, S9: Keyswitch, ScottoKeebs_Hotswap:Hotswap_Choc_V1V2_1.00u, symbol ScottoKeebs:Placeholder_Keyswitch
- added S31, S32, S33: Keyswitch, ScottoKeebs_Hotswap:Hotswap_Choc_V1V2_1.50u_90deg, symbol ScottoKeebs:Placeholder_Keyswitch
- D1, D2: footprint (none) -> ScottoKeebs_Components:Diode_SOD-123
- S1, S2: footprint (none) -> ScottoKeebs_Hotswap:Hotswap_Choc_V1V2_1.00u
- SW1: renamed from SW2; footprint (none) -> ScottoKeebs_Components:Button_MJTP1243
- SW2: renamed from SW1; footprint (none) -> Rotary_Encoder:RotaryEncoder_Alps_EC11E-Switch_Vertical_H20mm
- renumbered D12 to D98, U2 to U1, U1 to U2
Connections:
- net Col3: now reaches SW2.S1
- net Col3: now also S10.1, S16.1, S22.1, S4.1
- net at SW2.S2: now also D34.2 (A)
- net Row0: now reaches U1.3 (GP1)
- net Row0: now also D1.1 (K), D2.1 (K), D3.1 (K), D4.1 (K), D5.1 (K), D6.1 (K)
- net Col0: now reaches S1.1
- net Col0: now also S13.1, S19.1, S27.1, S7.1
- net Col1: now reaches S2.1
- net Col1: now also S14.1, S20.1, S28.1, S8.1
- new net: D9.2 (A), S9.2
- new net: D8.2 (A), S8.2
- new net: D29.2 (A), S29.2
- new net: D5.2 (A), S5.2
- new net: D32.2 (A), S32.2
- new net: D10.2 (A), S10.2
- new net: D25.2 (A), S25.2
- new net: D14.2 (A), S14.2
- new net: D23.2 (A), S23.2
- new net: D19.2 (A), S19.2
- new net: D17.2 (A), S17.2
- new net: D20.2 (A), S20.2
- new net: D4.2 (A), S4.2
- new net: D13.2 (A), S13.2
- new net: D11.2 (A), S11.2
- new net: D22.2 (A), S22.2
- new net: D12.2 (A), S12.2
- new net: D24.2 (A), S24.2
- new net: D6.2 (A), S6.2
- new net: D33.2 (A), S33.2
- new net: D18.2 (A), S18.2
- new net: D16.2 (A), S16.2
- new net: D21.2 (A), S21.2
- new net: D7.2 (A), S7.2
- new net: D15.2 (A), S15.2
- new net: D28.2 (A), S28.2
- new net: D31.2 (A), S31.2
- new net: D3.2 (A), S3.2
- new net: D26.2 (A), S26.2
- new net: D27.2 (A), S27.2
- new net: D30.2 (A), S30.2
- new net Col2: S15.1, S21.1, S29.1, S3.1, S9.1
- new net Col4: S11.1, S17.1, S23.1, S30.1, S5.1
- new net Col5: S12.1, S18.1, S24.1, S31.1, S6.1
- new net Col6: S25.1, S32.1
- new net Col7: S26.1, S33.1
- new net Row1: D10.1 (K), D11.1 (K), D12.1 (K), D7.1 (K), D8.1 (K), D9.1 (K)
- new net Row2: D13.1 (K), D14.1 (K), D15.1 (K), D16.1 (K), D17.1 (K), D18.1 (K)
- new net Row3: D19.1 (K), D20.1 (K), D21.1 (K), D22.1 (K), D23.1 (K), D24.1 (K), D25.1 (K), D26.1 (K)
- new net Row4: D27.1 (K), D28.1 (K), D29.1 (K), D30.1 (K), D31.1 (K), D32.1 (K), D33.1 (K), D34.1 (K)
Other:
- moved on the sheet: D2, D98, S2, SW2
